File: _autosave-Payload_Hardware_Schematic.kicad_sch (KiCad schematic)
At the start: 4 parts, among them J1 Micro_SD_Card, U1 STM32F411 BlackPill, U3 BMP388, U4 LSM9DS1

Commit message: updating full schematic
Connections:
- net GND: now also J1.1 (VSS); no longer J1.6 (VSS)
- net MISO2: now also J1.4 (DAT0/MISO); no longer J1.7 (DAT0/MISO)
- net MOSI2: now also J1.5 (DAT1/MOSI); no longer J1.8 (DAT1/MOSI)
- net SCK2: now also J1.3 (CLK); no longer J1.5 (CLK)
