File: _autosave-Payload_Hardware_Schematic.kicad_pcb (KiCad board)
At the start: 2 copper layers, 10 parts, among them J1 Micro_SD_Card, J2 Conn_01x06_Pin_5V, J3 Conn_01x06_Pin_3V3, J4 Conn_01x04_Pin, J5 Conn_01x08_Pin, U1 STM32F411 BlackPill, U2 MPM3610, U3 BMP388, U4 LSM9DS1, U5 MPM3610

Commit message: Editted power and labels
Parts:
- added U6: ~, Payload-BMP388:BMP388_Breakout, F.Cu at (123.1, 97.9)
Connections:
- J1 pad 9: (no net) -> unconnected-(J1-DET-Pad9)
