File: Payload_Hardware_Schematic.kicad_pcb (KiCad board)
At the start: 2 copper layers, 118 x 56 mm, 14 parts, among them J1 Micro_SD_Card, J3 Conn_01x04_Pin, J4 Conn_01x02, J5 Conn_01x04_Pin, J6 Conn_01x04_Socket, U1 STM32F411 BlackPill, U2 MPM3610, U4 LSM9DS1, U5 MPM3610, U6 BMP388

Commit message: Niv's edits, moved pins close to edge and connected servos to 7.2V
Parts:
- added J2: Conn_01x06_Socket, Connector_PinSocket_2.54mm:PinSocket_1x06_P2.54mm_Horizontal, F.Cu at (83.0, 100.0)
- moved J6 22.1 mm to (91.8, 78.6), turned to -90 degrees
- moved J1 17.0 mm to (96.4, 60.5)
Connections:
- J3 pad 3: /5V -> /7.2V
- J5 pad 3: /5V -> /7.2V
- U1 pad 20: unconnected-(U1-3.3V-Pad20) -> /<NO NET>
- U1 pad 21: /<NO NET> -> unconnected-(U1-VBat-Pad21)
Routing:
- net /SCK: track 22.7 -> 48.3 mm, vias 0 -> 1
- net /DIO: track 27.8 -> 52.4 mm, vias 0 -> 1
- net /<NO NET>: track 128.2 -> 106.9 mm, vias 0 -> 1
- net /MOSI2: track 26.7 -> 44.1 mm, vias 0 -> 1
- net /NSS2: track 12.6 -> 29.8 mm
- net /SCK2: track 9.34 -> 25.2 mm
- net /MISO2: track 26.7 -> 42.2 mm, vias 0 -> 1
- net /UART_TX: track 21.7 -> 35.3 mm
- net /UART_RX: track 24.5 -> 26.1 mm, vias 0 -> 1

Commit message: final gerber files
Parts:
- removed J6: Conn_01x04_Socket, Connector_PinHeader_2.54mm:PinHeader_1x04_P2.54mm_Horizontal
- moved J2 14.5 mm to (82.4, 85.5)
Routing:
- net /5V: track 41.2 -> 0.00 mm, vias 1 -> 0
- net /7.2V: track 27.8 -> 65.4 mm
- net /<NO NET>: track 106.9 -> 124.1 mm
- net /DIO: track 52.4 -> 61.8 mm
- net /SCK: track 48.3 -> 56.7 mm
- net /UART_RX: track 26.1 -> 34.2 mm
- net /UART_TX: track 35.3 -> 43.5 mm
- net /FDBK1: track 75.8 -> 77.1 mm
- net /SCK3: track 46.6 -> 47.5 mm
